Commit message: feat: Adjust B2+Z1 mount box size and position
- Reduced mount box height from 0.24m to 0.12m for lower profile
- Centered box geometry at mount point (extends -0.06 to +0.06)
- Updated Z1 attachment point to top of reduced box
- Adjusted launch file default z1_mount_x to 0.0 for center mounting
- Reduced box mass proportionally to 0.25kg

File: b2_z1_description/urdf/b2_z1.urdf.xacro (robot description, xacro)
@@ -13,5 +13,5 @@
     <!-- Z1 mounting position relative to B2 base_link (in meters) -->
     <!-- Default: slightly forward of center, above the body -->
-    <xacro:arg name="z1_mount_x" default="0.3" />    <!-- forward offset -->
+    <xacro:arg name="z1_mount_x" default="0.4" />    <!-- forward offset -->
     <xacro:arg name="z1_mount_y" default="0.0" />     <!-- lateral offset (0=center) -->
     <xacro:arg name="z1_mount_z" default="0.15" />    <!-- vertical offset above base -->
@@ -293,19 +293,19 @@
     <link name="z1_mount_box">
         <visual>
-            <origin xyz="0 0 0.05" rpy="0 0 0" />
+            <origin xyz="0 0 0" rpy="0 0 0" />
             <geometry>
-                <box size="0.12 0.15 0.24" />
+                <box size="0.12 0.15 0.12" />
             </geometry>
             <material name="Grey" />
         </visual>
         <collision>
-            <origin xyz="0 0 0.05" rpy="0 0 0" />
+            <origin xyz="0 0 0" rpy="0 0 0" />
             <geometry>
-                <box size="0.12 0.15 0.24" />
+                <box size="0.12 0.15 0.12" />
             </geometry>
         </collision>
         <inertial>
-            <origin xyz="0 0 0.05" rpy="0 0 0" />
-            <mass value="0.5" />
+            <origin xyz="0 0 0" rpy="0 0 0" />
+            <mass value="0.25" />
             <inertia ixx="0.002" ixy="0" ixz="0"
                      iyy="0.003" iyz="0"
@@ -324,5 +324,5 @@
         <parent link="z1_mount_box" />
         <child link="$(arg z1_prefix)link00" />
-        <origin xyz="0 0 0.1" rpy="0 0 0" />  <!-- Box height = 0.1m -->
+        <origin xyz="0 0 0.06" rpy="0 0 0" />  <!-- Half of 0.12m box above center -->
     </joint>
     <!-- Instantiate Z1 arm with prefix -->
